File: Dual-Mag-Camera-Control/COMMS.sch (KiCad schematic (older format))
At the start: 40 parts, among them J10 RS-232_2_3, J5 CVS-04TB, J6 CVS-04TB, J7 UART_0_1, J8 UART_2_3, J9 RS-232_0_1, U10 SparkFun_MAX3232, U9 SparkFun_MAX3232

Commit message: updated to KiCAD 6.0
Parts:
- D17, D18, D19, D20, D21, D22, D23, D24, D25, D26, D27, D28, D29, D30, D31, D32: symbol SPC-Control-rescue:D_TVS -> Dual-Mag-Camera-Control-rescue:D_TVS-SPC-Control-rescue
- F15, F16, F17, F18, F19, F20, F21, F22, F23, F24, F25, F26, F27, F28, F29, F30: symbol SPC-Control-rescue:Polyfuse_Small -> Dual-Mag-Camera-Control-rescue:Polyfuse_Small-SPC-Control-rescue
- J10, J7, J8, J9: symbol SPC-Control-rescue:Conn_01x06 -> Dual-Mag-Camera-Control-rescue:Conn_01x06-SPC-Control-rescue
- J5, J6: symbol SPC-Control-rescue:CVS-04TB -> Dual-Mag-Camera-Control-rescue:CVS-04TB-SPC-Control-rescue
- U10, U9: symbol ProjectDevices:SparkFun_MAX3232 -> Dual-Mag-Camera-Control-rescue:SparkFun_MAX3232-ProjectDevices
Changed lines of the file:
@@
 	7650 6900 7650 6800
 $Comp
-L SPC-Control-rescue:CVS-04TB J5
+L Dual-Mag-Camera-Control-rescue:CVS-04TB-SPC-Control-rescue J5
 U 1 1 5987E9DC
 P 4300 3450
@@
 UART_RX3
 $Comp
-L SPC-Control-rescue:CVS-04TB J6
+L Dual-Mag-Camera-Control-rescue:CVS-04TB-SPC-Control-rescue J6
 U 1 1 5A96228D
 P 8200 3450
@@
 $EndComp
 $Comp
-L SPC-Control-rescue:D_TVS D21
+L Dual-Mag-Camera-Control-rescue:D_TVS-SPC-Control-rescue D21
 U 1 1 5A96AB7C
 P 5700 4900
@@
 	9700 7150 10000 7150
 $Comp
-L SPC-Control-rescue:D_TVS D17
+L Dual-Mag-Camera-Control-rescue:D_TVS-SPC-Control-rescue D17
 U 1 1 604860DC
 P 4100 4900
@@
 $EndComp
 $Comp
-L SPC-Control-rescue:D_TVS D18
+L Dual-Mag-Camera-Control-rescue:D_TVS-SPC-Control-rescue D18
 U 1 1 60486583
 P 4100 5700
@@
 $EndComp
 $Comp
-L SPC-Control-rescue:D_TVS D19
+L Dual-Mag-Camera-Control-rescue:D_TVS-SPC-Control-rescue D19
 U 1 1 60486826
 P 4100 6650
@@
 $EndComp
 $Comp
-L SPC-Control-rescue:D_TVS D20
+L Dual-Mag-Camera-Control-rescue:D_TVS-SPC-Control-rescue D20
 U 1 1 60486CA1
 P 4100 7450
@@
 $EndComp
 $Comp
-L SPC-Control-rescue:D_TVS D24
+L Dual-Mag-Camera-Control-rescue:D_TVS-SPC-Control-rescue D24
 U 1 1 60486F78
 P 5700 7450
@@
 $EndComp
 $Comp
-L SPC-Control-rescue:D_TVS D23
+L Dual-Mag-Camera-Control-rescue:D_TVS-SPC-Control-rescue D23
 U 1 1 60487277
 P 5700 6650
@@
 $EndComp
 $Comp
-L SPC-Control-rescue:D_TVS D22
+L Dual-Mag-Camera-Control-rescue:D_TVS-SPC-Control-rescue D22
 U 1 1 604875E8
 P 5700 5700
@@
 $EndComp
 $Comp
-L SPC-Control-rescue:Polyfuse_Small F28
+L Dual-Mag-Camera-Control-rescue:Polyfuse_Small-SPC-Control-rescue F28
 U 1 1 60489A8C
 P 9450 5400
@@
 $EndComp
 $Comp
-L SPC-Control-rescue:Polyfuse_Small F29
+L Dual-Mag-Camera-Control-rescue:Polyfuse_Small-SPC-Control-rescue F29
 U 1 1 60489E29
 P 9450 6350
@@
 $EndComp
 $Comp
-L SPC-Control-rescue:Polyfuse_Small F30
+L Dual-Mag-Camera-Control-rescue:Polyfuse_Small-SPC-Control-rescue F30
 U 1 1 6048A0D2
 P 9450 7150
@@
 $EndComp
 $Comp
-L SPC-Control-rescue:Polyfuse_Small F26
+L Dual-Mag-Camera-Control-rescue:Polyfuse_Small-SPC-Control-rescue F26
 U 1 1 6048A483
 P 7400 7150
@@
 $EndComp
 $Comp
-L SPC-Control-rescue:Polyfuse_Small F25
+L Dual-Mag-Camera-Control-rescue:Polyfuse_Small-SPC-Control-rescue F25
 U 1 1 6048A9E0
 P 7400 6350
@@
 $EndComp
 $Comp
-L SPC-Control-rescue:Polyfuse_Small F24
+L Dual-Mag-Camera-Control-rescue:Polyfuse_Small-SPC-Control-rescue F24
 U 1 1 6048AD7D
 P 7400 5400
@@
 $EndComp
 $Comp
-L SPC-Control-rescue:Polyfuse_Small F23
+L Dual-Mag-Camera-Control-rescue:Polyfuse_Small-SPC-Control-rescue F23
 U 1 1 6048B16A
 P 7400 4600
@@
 $EndComp
 $Comp
-L SPC-Control-rescue:Polyfuse_Small F19
+L Dual-Mag-Camera-Control-rescue:Polyfuse_Small-SPC-Control-rescue F19
 U 1 1 6048B52F
 P 5450 4600
@@
 $EndComp
 $Comp
-L SPC-Control-rescue:Polyfuse_Small F21
+L Dual-Mag-Camera-Control-rescue:Polyfuse_Small-SPC-Control-rescue F21
 U 1 1 6048B980
 P 5450 6350
@@
 $EndComp
 $Comp
-L SPC-Control-rescue:Polyfuse_Small F20
+L Dual-Mag-Camera-Control-rescue:Polyfuse_Small-SPC-Control-rescue F20
 U 1 1 6048BFB1
 P 5450 5400
@@
 $EndComp
 $Comp
-L SPC-Control-rescue:Polyfuse_Small F22
+L Dual-Mag-Camera-Control-rescue:Polyfuse_Small-SPC-Control-rescue F22
 U 1 1 6048C26A
 P 5450 7150
@@
 $EndComp
 $Comp
-L SPC-Control-rescue:Polyfuse_Small F18
+L Dual-Mag-Camera-Control-rescue:Polyfuse_Small-SPC-Control-rescue F18
 U 1 1 6048C573
 P 3850 7150
@@
 $EndComp
 $Comp
-L SPC-Control-rescue:Polyfuse_Small F17
+L Dual-Mag-Camera-Control-rescue:Polyfuse_Small-SPC-Control-rescue F17
 U 1 1 6048C95C
 P 3850 6350
@@
 $EndComp
 $Comp
-L SPC-Control-rescue:Polyfuse_Small F16
+L Dual-Mag-Camera-Control-rescue:Polyfuse_Small-SPC-Control-rescue F16
 U 1 1 6048CCCD
 P 3850 5400
@@
 $EndComp
 $Comp
-L SPC-Control-rescue:Polyfuse_Small F15
+L Dual-Mag-Camera-Control-rescue:Polyfuse_Small-SPC-Control-rescue F15
 U 1 1 6048D0DE
 P 3850 4600
@@
 $EndComp
 $Comp
-L ProjectDevices:SparkFun_MAX3232 U9
+L Dual-Mag-Camera-Control-rescue:SparkFun_MAX3232-ProjectDevices U9
 U 1 1 604E6489
 P 5300 3150
@@
 	5000 3100 4900 3100
 $Comp
-L ProjectDevices:SparkFun_MAX3232 U10
+L Dual-Mag-Camera-Control-rescue:SparkFun_MAX3232-ProjectDevices U10
 U 1 1 60560389
 P 9400 3150
@@
 	9700 4600 10000 4600
 $Comp
-L SPC-Control-rescue:Polyfuse_Small F27
+L Dual-Mag-Camera-Control-rescue:Polyfuse_Small-SPC-Control-rescue F27
 U 1 1 59887D80
 P 9450 4600
@@
 	12600 7850 12750 7850
 $Comp
-L SPC-Control-rescue:D_TVS D?
+L Dual-Mag-Camera-Control-rescue:D_TVS-SPC-Control-rescue D?
 U 1 1 602E29BE
 P 7650 4900
@@
 $EndComp
 $Comp
-L SPC-Control-rescue:D_TVS D?
+L Dual-Mag-Camera-Control-rescue:D_TVS-SPC-Control-rescue D?
 U 1 1 602E8DB6
 P 9700 4900
@@
 $EndComp
 $Comp
-L SPC-Control-rescue:D_TVS D?
+L Dual-Mag-Camera-Control-rescue:D_TVS-SPC-Control-rescue D?
 U 1 1 602E920B
 P 9700 5700
@@
 $EndComp
 $Comp
-L SPC-Control-rescue:D_TVS D?
+L Dual-Mag-Camera-Control-rescue:D_TVS-SPC-Control-rescue D?
 U 1 1 602E961C
 P 7650 5700
@@
 $EndComp
 $Comp
-L SPC-Control-rescue:D_TVS D?
+L Dual-Mag-Camera-Control-rescue:D_TVS-SPC-Control-rescue D?
 U 1 1 602E9B7B
 P 7650 6650
@@
 $EndComp
 $Comp
-L SPC-Control-rescue:D_TVS D?
+L Dual-Mag-Camera-Control-rescue:D_TVS-SPC-Control-rescue D?
 U 1 1 602E9F66
 P 9700 6650
@@
 $EndComp
 $Comp
-L SPC-Control-rescue:D_TVS D?
+L Dual-Mag-Camera-Control-rescue:D_TVS-SPC-Control-rescue D?
 U 1 1 602EA2A9
 P 9700 7450
@@
 $EndComp
 $Comp
-L SPC-Control-rescue:D_TVS D?
+L Dual-Mag-Camera-Control-rescue:D_TVS-SPC-Control-rescue D?
 U 1 1 602EA6FC
 P 7650 7450
@@
 $EndComp
 $Comp
-L SPC-Control-rescue:Conn_01x06 J?
+L Dual-Mag-Camera-Control-rescue:Conn_01x06-SPC-Control-rescue J?
 U 1 1 60356825
 P 12950 4800
@@
 $EndComp
 $Comp
-L SPC-Control-rescue:Conn_01x06 J?
+L Dual-Mag-Camera-Control-rescue:Conn_01x06-SPC-Control-rescue J?
 U 1 1 6035D2B9
 P 12950 5700
@@
 $EndComp
 $Comp
-L SPC-Control-rescue:Conn_01x06 J?
+L Dual-Mag-Camera-Control-rescue:Conn_01x06-SPC-Control-rescue J?
 U 1 1 6035D8FE
 P 12950 6600
@@
 $EndComp
 $Comp
-L SPC-Control-rescue:Conn_01x06 J?
+L Dual-Mag-Camera-Control-rescue:Conn_01x06-SPC-Control-rescue J?
 U 1 1 6035DDE7
 P 12950 7550
