File: Dual-Mag-Camera-Control/CameraPower.sch (KiCad schematic (older format))
At the start: 4 parts, among them U11 S18V20F12, U12 S18V20F12

Commit message: updated to KiCAD 6.0
Parts:
- U11, U12: symbol ProjectDevices:S18V20F12 -> Dual-Mag-Camera-Control-rescue:S18V20F12-ProjectDevices
Changed lines of the file:
@@
 $EndDescr
 $Comp
-L ProjectDevices:S18V20F12 U?
+L Dual-Mag-Camera-Control-rescue:S18V20F12-ProjectDevices U?
 U 1 1 5F4AAE3D
 P 7450 4700
@@
 	10300 5450 10300 5950
 $Comp
-L ProjectDevices:S18V20F12 U?
+L Dual-Mag-Camera-Control-rescue:S18V20F12-ProjectDevices U?
 U 1 1 5F709A19
 P 7450 5650
