File: Dual-Mag-Camera-Control/Dual-Mag-Camera-Control.kicad_pcb (KiCad board)
At the start: 2 copper layers, 152.4 x 96.5 mm, 144 parts, among them J1 ~TRIG_IO, J10 RS-232_2_3, J11 PWR_IN_1, J12 PWR_IN_2, J13 STRB_PWR, J14 CAM_COMPUTE_PWR, J15 5V_5A_PWR, J16 5V_2.5A_PWR, J2 TRIG_IO, J3 ADC_DAC, J4 GPIO, J5 CVS-04TB, J6 CVS-04TB, J7 UART_0_1, J8 UART_2_3, J9 RS-232_0_1, Q1 Si7463DP, Q2 Si7463DP, Q3 Si7463DP, Q4 Si7463DP, Q5 SISS10ADN, Q6 SI7611DN, Q7 SISS10ADN, Q8 SI7611DN, Q9 Si7463DP, U1 D24V10F5, U10 SparkFun_MAX3232, U11 S18V20F12, U12 S18V20F12, U13 LTC4412HVIS6, U14 LTC4412HVIS6, U15 LTC4412HVIS6, U16 LTC4412HVIS6, U17 LTC4412HVIS6, U2 Adafruit_BME280, U3 D24V50F5, U4 LowPowerLab-SD-Card, U5 D24V22F5, U6 Adafruit_INA260, U7 Adafruit_INA260, U8 MoteinoM0, U9 SparkFun_MAX3232

Commit message: updated to KiCAD 6.0
Parts:
- J1: value ~TRIG_IO -> ~{TRIG_IO}
Connections:
- net /~12V_ENABLE renamed /~{12V_ENABLE}
- net /~5V_ENABLE renamed /~{5V_ENABLE}
- net /~STROBE_ENABLE renamed /~{STROBE_ENABLE}
Other:
- outline, holes or cut-outs redrawn
- net class Default removed
