File: Dual-Mag-Camera-Control/Dual-Mag-Camera-Control.sch (KiCad schematic (older format))
At the start: 55 parts, among them J1 ~TRIG_IO, J11 PWR_IN_1, J12 PWR_IN_2, J13 STRB_PWR, J14 CAM_COMPUTE_PWR, J15 5V_5A_PWR, J16 5V_2.5A_PWR, J2 TRIG_IO, J3 ADC_DAC, J4 GPIO, U1 D24V10F5, U2 Adafruit_BME280, U3 D24V50F5, U4 LowPowerLab-SD-Card, U5 D24V22F5, U6 Adafruit_INA260, U7 Adafruit_INA260, U8 MoteinoM0

Commit message: updated to KiCAD 6.0
Parts:
- D10, D11, D12, D13, D14, D15, D16, D4, D5, D6, D7, D8, D9: symbol SPC-Control-rescue:D_TVS -> Dual-Mag-Camera-Control-rescue:D_TVS-SPC-Control-rescue
- F10, F11, F12, F13, F14, F2, F3, F4, F5, F6, F7, F8, F9: symbol SPC-Control-rescue:Polyfuse_Small -> Dual-Mag-Camera-Control-rescue:Polyfuse_Small-SPC-Control-rescue
- J1, J2, J3, J4: symbol SPC-Control-rescue:Conn_01x06 -> Dual-Mag-Camera-Control-rescue:Conn_01x06-SPC-Control-rescue
- R19, R20: symbol BUMP-Control-rescue:Resistor_small-SPC-Control-rescue-DeathStar-rescue -> Dual-Mag-Camera-Control-rescue:Resistor_small-SPC-Control-rescue-DeathStar-rescue-BUMP-Control-rescue
- U1: symbol ProjectDevices:D24V10F5 -> Dual-Mag-Camera-Control-rescue:D24V10F5-ProjectDevices
- U2: symbol ProjectDevices:Adafruit_BME280 -> Dual-Mag-Camera-Control-rescue:Adafruit_BME280-ProjectDevices
- U3: symbol ProjectDevices:D24V50F5 -> Dual-Mag-Camera-Control-rescue:D24V50F5-ProjectDevices
- U4: symbol ProjectDevices:LowPowerLab-SD-Card -> Dual-Mag-Camera-Control-rescue:LowPowerLab-SD-Card-ProjectDevices
- U5: symbol ProjectDevices:D24V22F5 -> Dual-Mag-Camera-Control-rescue:D24V22F5-ProjectDevices
- U6, U7: symbol ProjectDevices:Adafruit_INA260 -> Dual-Mag-Camera-Control-rescue:Adafruit_INA260-ProjectDevices
Changed lines of the file:
@@
 $EndSheet
 $Comp
-L ProjectDevices:D24V10F5 U1
+L Dual-Mag-Camera-Control-rescue:D24V10F5-ProjectDevices U1
 U 1 1 5F4F2D79
 P 2200 4750
@@
 GND
 $Comp
-L ProjectDevices:Adafruit_INA260 U6
+L Dual-Mag-Camera-Control-rescue:Adafruit_INA260-ProjectDevices U6
 U 1 1 5FA2716F
 P 7150 1600
@@
 Power Input Protection, Ideal Diodes, and Monitoring\n\n
 $Comp
-L ProjectDevices:Adafruit_BME280 U2
+L Dual-Mag-Camera-Control-rescue:Adafruit_BME280-ProjectDevices U2
 U 1 1 5F5548D0
 P 2250 7750
@@
 TTL and RS-232 COMMS\n\n
 $Comp
-L ProjectDevices:D24V50F5 U3
+L Dual-Mag-Camera-Control-rescue:D24V50F5-ProjectDevices U3
 U 1 1 6023F0CB
 P 4700 5900
@@
 $EndComp
 $Comp
-L ProjectDevices:D24V22F5 U5
+L Dual-Mag-Camera-Control-rescue:D24V22F5-ProjectDevices U5
 U 1 1 6024AA7C
 P 6200 5900
@@
 ~STROBE_ENABLE
 $Comp
-L SPC-Control-rescue:Polyfuse_Small F?
+L Dual-Mag-Camera-Control-rescue:Polyfuse_Small-SPC-Control-rescue F?
 U 1 1 5F905C4F
 P 13450 5500
@@
 	13250 5950 13700 5950
 $Comp
-L SPC-Control-rescue:Polyfuse_Small F?
+L Dual-Mag-Camera-Control-rescue:Polyfuse_Small-SPC-Control-rescue F?
 U 1 1 5F932284
 P 13450 4850
@@
 	13250 5300 13700 5300
 $Comp
-L SPC-Control-rescue:Polyfuse_Small F?
+L Dual-Mag-Camera-Control-rescue:Polyfuse_Small-SPC-Control-rescue F?
 U 1 1 5F93E769
 P 15150 5500
@@
 $EndComp
 $Comp
-L SPC-Control-rescue:D_TVS D?
+L Dual-Mag-Camera-Control-rescue:D_TVS-SPC-Control-rescue D?
 U 1 1 5F93E776
 P 15400 5700
@@
 	14950 5950 15400 5950
 $Comp
-L SPC-Control-rescue:Polyfuse_Small F?
+L Dual-Mag-Camera-Control-rescue:Polyfuse_Small-SPC-Control-rescue F?
 U 1 1 5F93E78D
 P 15150 4850
@@
 	14950 5300 15400 5300
 $Comp
-L SPC-Control-rescue:Polyfuse_Small F?
+L Dual-Mag-Camera-Control-rescue:Polyfuse_Small-SPC-Control-rescue F?
 U 1 1 5F94C855
 P 11750 5500
@@
 	11550 5950 12000 5950
 $Comp
-L SPC-Control-rescue:Polyfuse_Small F?
+L Dual-Mag-Camera-Control-rescue:Polyfuse_Small-SPC-Control-rescue F?
 U 1 1 5F94C879
 P 11750 4850
@@
 	4750 6350 4950 6350
 $Comp
-L SPC-Control-rescue:D_TVS D?
+L Dual-Mag-Camera-Control-rescue:D_TVS-SPC-Control-rescue D?
 U 1 1 5F8B199B
 P 15400 5050
@@
 $EndComp
 $Comp
-L SPC-Control-rescue:D_TVS D?
+L Dual-Mag-Camera-Control-rescue:D_TVS-SPC-Control-rescue D?
 U 1 1 5F8B1E18
 P 13700 5050
@@
 $EndComp
 $Comp
-L SPC-Control-rescue:D_TVS D?
+L Dual-Mag-Camera-Control-rescue:D_TVS-SPC-Control-rescue D?
 U 1 1 5F8B2281
 P 13700 5700
@@
 $EndComp
 $Comp
-L SPC-Control-rescue:D_TVS D?
+L Dual-Mag-Camera-Control-rescue:D_TVS-SPC-Control-rescue D?
 U 1 1 5F8B271E
 P 12000 5700
@@
 $EndComp
 $Comp
-L SPC-Control-rescue:D_TVS D?
+L Dual-Mag-Camera-Control-rescue:D_TVS-SPC-Control-rescue D?
 U 1 1 5F8B2C5B
 P 12000 5050
@@
 	13700 4700 13700 4850
 $Comp
-L SPC-Control-rescue:Polyfuse_Small F?
+L Dual-Mag-Camera-Control-rescue:Polyfuse_Small-SPC-Control-rescue F?
 U 1 1 5F922860
 P 11750 6150
@@
 $EndComp
 $Comp
-L SPC-Control-rescue:D_TVS D?
+L Dual-Mag-Camera-Control-rescue:D_TVS-SPC-Control-rescue D?
 U 1 1 5F92286D
 P 12000 6350
@@
 	11550 6600 12000 6600
 $Comp
-L SPC-Control-rescue:Polyfuse_Small F?
+L Dual-Mag-Camera-Control-rescue:Polyfuse_Small-SPC-Control-rescue F?
 U 1 1 5F97EDEE
 P 13450 6150
@@
 $EndComp
 $Comp
-L SPC-Control-rescue:D_TVS D?
+L Dual-Mag-Camera-Control-rescue:D_TVS-SPC-Control-rescue D?
 U 1 1 5F97EDFB
 P 13700 6350
@@
 	13250 6600 13700 6600
 $Comp
-L SPC-Control-rescue:Polyfuse_Small F?
+L Dual-Mag-Camera-Control-rescue:Polyfuse_Small-SPC-Control-rescue F?
 U 1 1 5F9900D3
 P 15150 6150
@@
 $EndComp
 $Comp
-L SPC-Control-rescue:D_TVS D?
+L Dual-Mag-Camera-Control-rescue:D_TVS-SPC-Control-rescue D?
 U 1 1 5F9900E0
 P 15400 6350
@@
 	14950 6600 15400 6600
 $Comp
-L SPC-Control-rescue:Polyfuse_Small F?
+L Dual-Mag-Camera-Control-rescue:Polyfuse_Small-SPC-Control-rescue F?
 U 1 1 5F9A24DA
 P 11750 6800
@@
 $EndComp
 $Comp
-L SPC-Control-rescue:D_TVS D?
+L Dual-Mag-Camera-Control-rescue:D_TVS-SPC-Control-rescue D?
 U 1 1 5F9A24E7
 P 12000 7000
@@
 	11550 7250 12000 7250
 $Comp
-L SPC-Control-rescue:Polyfuse_Small F?
+L Dual-Mag-Camera-Control-rescue:Polyfuse_Small-SPC-Control-rescue F?
 U 1 1 5F9CA406
 P 13450 6800
@@
 $EndComp
 $Comp
-L SPC-Control-rescue:D_TVS D?
+L Dual-Mag-Camera-Control-rescue:D_TVS-SPC-Control-rescue D?
 U 1 1 5F9CA413
 P 13700 7000
@@
 	13250 7250 13700 7250
 $Comp
-L SPC-Control-rescue:Polyfuse_Small F?
+L Dual-Mag-Camera-Control-rescue:Polyfuse_Small-SPC-Control-rescue F?
 U 1 1 5F9F1679
 P 15150 6800
@@
 $EndComp
 $Comp
-L SPC-Control-rescue:D_TVS D?
+L Dual-Mag-Camera-Control-rescue:D_TVS-SPC-Control-rescue D?
 U 1 1 5F9F1686
 P 15400 7000
@@
 	14950 7250 15400 7250
 $Comp
-L SPC-Control-rescue:Conn_01x06 J1
+L Dual-Mag-Camera-Control-rescue:Conn_01x06-SPC-Control-rescue J1
 U 1 1 5FA8C201
 P 13400 7950
@@
 GND
 $Comp
-L ProjectDevices:LowPowerLab-SD-Card U4
+L Dual-Mag-Camera-Control-rescue:LowPowerLab-SD-Card-ProjectDevices U4
 U 1 1 5FC64C34
 P 5100 7850
@@
 DAC_OUT_IO
 $Comp
-L SPC-Control-rescue:Polyfuse_Small F?
+L Dual-Mag-Camera-Control-rescue:Polyfuse_Small-SPC-Control-rescue F?
 U 1 1 5FE8693A
 P 11950 7750
@@
 $EndComp
 $Comp
-L SPC-Control-rescue:D_TVS D?
+L Dual-Mag-Camera-Control-rescue:D_TVS-SPC-Control-rescue D?
 U 1 1 5FE86947
 P 12200 7950
@@
 	13100 8250 13200 8250
 $Comp
-L ProjectDevices:Adafruit_INA260 U7
+L Dual-Mag-Camera-Control-rescue:Adafruit_INA260-ProjectDevices U7
 U 1 1 60321937
 P 9200 2850
@@
 $EndComp
 $Comp
-L SPC-Control-rescue:Conn_01x06 J2
+L Dual-Mag-Camera-Control-rescue:Conn_01x06-SPC-Control-rescue J2
 U 1 1 60353CE5
 P 14300 7950
@@
 $EndComp
 $Comp
-L SPC-Control-rescue:Conn_01x06 J3
+L Dual-Mag-Camera-Control-rescue:Conn_01x06-SPC-Control-rescue J3
 U 1 1 60354316
 P 15100 7950
@@
 $EndComp
 $Comp
-L SPC-Control-rescue:Conn_01x06 J4
+L Dual-Mag-Camera-Control-rescue:Conn_01x06-SPC-Control-rescue J4
 U 1 1 6035491B
 P 15900 7950
@@
 $EndComp
 $Comp
-L BUMP-Control-rescue:Resistor_small-SPC-Control-rescue-DeathStar-rescue R?
+L Dual-Mag-Camera-Control-rescue:Resistor_small-SPC-Control-rescue-DeathStar-rescue-BUMP-Control-rescue R?
 U 1 1 605B43FE
 P 11850 3250
@@
 	11850 3450 11850 3350
 $Comp
-L BUMP-Control-rescue:Resistor_small-SPC-Control-rescue-DeathStar-rescue R?
+L Dual-Mag-Camera-Control-rescue:Resistor_small-SPC-Control-rescue-DeathStar-rescue-BUMP-Control-rescue R?
 U 1 1 605CABF5
 P 11550 3250
