File: Dual-Mag-Camera-Control/HighSideSwitch_LTC4412HV.sch (KiCad schematic (older format))
At the start: 5 parts, among them Q9 Si7463DP, U17 LTC4412HVIS6

Commit message: updated to KiCAD 6.0
Parts:
- Q9: symbol ProjectDevices:Si7463DP -> Dual-Mag-Camera-Control-rescue:Si7463DP-ProjectDevices
Changed lines of the file:
@@
 NoConn ~ 5850 3850
 $Comp
-L ProjectDevices:Si7463DP Q?
+L Dual-Mag-Camera-Control-rescue:Si7463DP-ProjectDevices Q?
 U 1 1 606003DC
 P 5400 3000
