File: Dual-Mag-Camera-Control/LTC4412HV.sch (KiCad schematic (older format))
At the start: 6 parts, among them Q1 Si7463DP, U13 LTC4412HVIS6

Commit message: updated to KiCAD 6.0
Parts:
- Q1: symbol ProjectDevices:Si7463DP -> Dual-Mag-Camera-Control-rescue:Si7463DP-ProjectDevices
Changed lines of the file:
@@
 $EndComp
 $Comp
-L ProjectDevices:Si7463DP Q?
+L Dual-Mag-Camera-Control-rescue:Si7463DP-ProjectDevices Q?
 U 1 1 5F4BCBD6
 P 7600 4500
