File: Dual-Mag-Camera-Control/PowerInputProtection.sch (KiCad schematic (older format))
At the start: 8 parts, among them Q5 SISS10ADN, Q6 SI7611DN

Commit message: updated to KiCAD 6.0
Parts:
- removed Q6: SI7611DN, Package_SO:Vishay_PowerPAK_1212-8_Single, symbol SPC-Control-rescue:SiS443DN
- added Q?: Si7463DP, Package_SO:PowerPAK_SO-8_Single, symbol Dual-Mag-Camera-Control-rescue:Si7463DP-ProjectDevices
- C9: symbol SPC-Control-rescue:C_Small -> Dual-Mag-Camera-Control-rescue:C_Small-SPC-Control-rescue
- D34: symbol BUMP-Control-rescue:ZENERsmall-RESCUE-PowerControlBoard-SPC-Control-rescue-DeathStar-rescue -> Dual-Mag-Camera-Control-rescue:ZENERsmall-RESCUE-PowerControlBoard-SPC-Control-rescue-DeathStar-rescue-BUMP-Control-res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
- F1: symbol ProjectDevices:01550900M(Holder) -> Dual-Mag-Camera-Control-rescue:01550900M(Holder)-ProjectDevices
- Q5: value SISS10ADN -> SISS12DN; symbol ProjectDevices:SiSA72DN -> Dual-Mag-Camera-Control-rescue:SiSA72DN-ProjectDevices; Link https://www.digikey.com/product-detail/en/vishay-siliconix/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 -> https://www.digikey.com/en/products/detail/vishay-siliconix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; Part Number SISS10ADN-T1-GE3 -> SISS12DN-T1-GE3CT-ND
- R12: symbol BUMP-Control-rescue:Resistor_small-SPC-Control-rescue-DeathStar-rescue -> Dual-Mag-Camera-Control-rescue:Resistor_small-SPC-Control-rescue-DeathStar-rescue-BUMP-Control-rescue
- R13, R14: symbol SPC-Control-rescue:Resistor_small -> Dual-Mag-Camera-Control-rescue:Resistor_small-SPC-Control-rescue
Connections:
- net Vout: now also Q?.5 (D)
- net at R13.1, R14.1: now also Q?.4 (G)
- net at C9.1, F1.2, R12.1: now also Q?.1 (S), Q?.2 (S), Q?.3 (S)
Changed lines of the file:
@@
 $Descr B 17000 11000
 encoding utf-8
-Sheet 9 10
+Sheet 8 10
 Title "PowerInputProtection"
 Date "2020-09-19"
@@
 Reverse Polairty Protection
 $Comp
-L ProjectDevices:01550900M(Holder) F1
+L Dual-Mag-Camera-Control-rescue:01550900M(Holder)-ProjectDevices F1
 U 1 1 607CC1EA
 P 6850 4400
 AR Path="/5F7C3A84/607CC1EA" Ref="F1"  Part="1"
 AR Path="/5F81819E/607CC1EA" Ref="F31"  Part="1"
-F 0 "F31" H 6850 4615 50  0000 C CNN
+F 0 "F1" H 6850 4615 50  0000 C CNN
 F 1 "01550900M(Holder)" H 6850 4524 50  0000 C CNN
 F 2 "ProjectFootprints:01550900M" H 6800 3950 50  0001 C CNN
@@
 $EndComp
 $Comp
-L ProjectDevices:SiSA72DN Q?
+L Dual-Mag-Camera-Control-rescue:SiSA72DN-ProjectDevices Q?
 U 1 1 6039125F
 P 7150 5500
@@
 AR Path="/5F7C3A84/6039125F" Ref="Q5"  Part="1"
 AR Path="/5F81819E/6039125F" Ref="Q7"  Part="1"
-F 0 "Q7" V 6950 5550 50  0000 C CNN
-F 1 "SISS10ADN" V 6850 5700 50  0000 C CNN
+F 0 "Q5" V 6950 5550 50  0000 C CNN
+F 1 "SISS12DN" V 6850 5700 50  0000 C CNN
 F 2 "Package_SO:Vishay_PowerPAK_1212-8_Single" H 7150 5500 50  0001 C CNN
-F 3 "https://www.vishay.com/docs/79237/siss10adn.pdf" H 7150 5500 50  0001 C CNN
-F 4 "SISS10ADN-T1-GE3" H 7150 5500 50  0001 C CNN "Part Number"
+F 3 "https://www.vishay.com/docs/75281/siss12dn.pdf" H 7150 5500 50  0001 C CNN
+F 4 "SISS12DN-T1-GE3CT-ND" H 7150 5500 50  0001 C CNN "Part Number"
 F 5 "Digikey" H 7150 5500 50  0001 C CNN "Supplier"
-F 6 "https://www.digikey.com/product-detail/en/vishay-siliconix/SISS10ADN-T1-GE3/SISS10ADN-T1-GE3CT-ND/9760611" H 7150 5500 50  0001 C CNN "Link"
+F 6 "https://www.digikey.com/en/products/detail/vishay-siliconix/siss12dn-t1-ge3/8572063" H 7150 5500 50  0001 C CNN "Link"
 	1    7150 5500
 	0    -1   1    0
 $EndComp
 $Comp
-L BUMP-Control-rescue:ZENERsmall-RESCUE-PowerControlBoard-SPC-Control-rescue-DeathStar-rescue D?
+L Dual-Mag-Camera-Control-rescue:ZENERsmall-RESCUE-PowerControlBoard-SPC-Control-rescue-DeathStar-rescue-BUMP-Control-rescue D?
 U 1 1 60391260
 P 7850 5000
@@
 AR Path="/5F7C3A84/60391260" Ref="D34"  Part="1"
 AR Path="/5F81819E/60391260" Ref="D35"  Part="1"
-F 0 "D35" V 7750 4850 50  0000 C CNN
+F 0 "D34" V 7750 4850 50  0000 C CNN
 F 1 "BZT52C20T-7" V 7850 4650 50  0000 C CNN
 F 2 "Diode_SMD:D_SOD-523" H 7850 5000 50  0001 C CNN
@@
 $EndComp
 $Comp
-L BUMP-Control-rescue:Resistor_small-SPC-Control-rescue-DeathStar-rescue R?
+L Dual-Mag-Camera-Control-rescue:Resistor_small-SPC-Control-rescue-DeathStar-rescue-BUMP-Control-rescue R?
 U 1 1 60391261
 P 7850 4600
@@
 AR Path="/5F7C3A84/60391261" Ref="R12"  Part="1"
 AR Path="/5F81819E/60391261" Ref="R15"  Part="1"
-F 0 "R15" H 7750 4650 50  0000 C CNN
+F 0 "R12" H 7750 4650 50  0000 C CNN
 F 1 "10K" H 7700 4550 50  0000 C CNN
 F 2 "Resistor_SMD:R_0603_1608Metric_Pad1.05x0.95mm_HandSolder" V 7780 4600 50  0001 C CNN
@@
 	7850 4800 7850 4700
 $Comp
-L SPC-Control-rescue:SiS443DN Q?
-U 1 1 6039125E
-P 9450 4550
-AR Path="/5A8F9077/6039125E" Ref="Q?"  Part="1"
-AR Path="/5F4E7452/6039125E" Ref="Q?"  Part="1"
-AR Path="/5F484405/6039125E" Ref="Q?"  Part="1"
-AR Path="/5F7C3A84/6039125E" Ref="Q6"  Part="1"
-AR Path="/5F81819E/6039125E" Ref="Q8"  Part="1"
-AR Path="/6039125E" Ref="Q?"  Part="1"
-F 0 "Q8" V 9800 4650 50  0000 L CNN
-F 1 "SI7611DN" V 9800 4200 50  0000 L CNN
-F 2 "Package_SO:Vishay_PowerPAK_1212-8_Single" H 9825 4450 50  0001 L CNN
-F 3 "https://www.vishay.com/docs/69939/si7611dn.pdf" H 9450 4550 50  0001 L CNN
-F 4 "SI7611DN-T1-GE3" H 9450 4550 60  0001 C CNN "Part Number"
-F 5 "Digikey" H 9450 4550 60  0001 C CNN "Supplier"
-F 6 "https://www.digikey.com/product-detail/en/vishay-siliconix/SI7611DN-T1-GE3/SI7611DN-T1-GE3CT-ND/1978912" H 9450 4550 60  0001 C CNN "Link"
-	1    9450 4550
-	0    1    -1   0
-$EndComp
-$Comp
-L SPC-Control-rescue:Resistor_small R?
+L Dual-Mag-Camera-Control-rescue:Resistor_small-SPC-Control-rescue R?
 U 1 1 5F7D2C57
 P 9100 4750
@@
 AR Path="/5F81819E/5F7D2C57" Ref="R16"  Part="1"
 AR Path="/5F7D2C57" Ref="R?"  Part="1"
-F 0 "R16" V 9180 4750 50  0000 C CNN
+F 0 "R13" V 9180 4750 50  0000 C CNN
 F 1 "100" V 9020 4760 50  0000 C CNN
 F 2 "Resistor_SMD:R_0603_1608Metric" V 9030 4750 50  0001 C CNN
@@
 $EndComp
 $Comp
-L SPC-Control-rescue:Resistor_small R?
+L Dual-Mag-Camera-Control-rescue:Resistor_small-SPC-Control-rescue R?
 U 1 1 60391263
 P 9400 5050
@@
 AR Path="/5F81819E/60391263" Ref="R17"  Part="1"
 AR Path="/60391263" Ref="R?"  Part="1"
-F 0 "R17" V 9480 5050 50  0000 C CNN
+F 0 "R14" V 9480 5050 50  0000 C CNN
 F 1 "499k" V 9320 5060 50  0000 C CNN
 F 2 "Resistor_SMD:R_0603_1608Metric" V 9330 5050 50  0001 C CNN
@@
 $EndComp
 Wire Wire Line
-	9250 4400 9250 4350
-Connection ~ 9250 4350
-Wire Wire Line
 	8700 4400 8700 4550
 Connection ~ 8700 4400
@@
 	9400 4600 9400 4750
 Connection ~ 9400 4750
-Wire Wire Line
-	9650 4300 9650 4350
-Connection ~ 9650 4350
 Connection ~ 9650 4400
 $Comp
-L SPC-Control-rescue:C_Small C?
+L Dual-Mag-Camera-Control-rescue:C_Small-SPC-Control-rescue C?
 U 1 1 5F7D2C5A
 P 8700 4650
@@
 AR Path="/5F81819E/5F7D2C5A" Ref="C10"  Part="1"
 AR Path="/5F7D2C5A" Ref="C?"  Part="1"
-F 0 "C10" H 8800 4750 50  0000 L CNN
+F 0 "C9" H 8800 4750 50  0000 L CNN
 F 1 "1 uF" H 8800 4650 50  0000 L CNN
 F 2 "Capacitor_SMD:C_0805_2012Metric" H 8700 4650 50  0001 C CNN
@@
 $EndComp
 Wire Wire Line
-	9250 4350 9250 4300
-Wire Wire Line
 	8700 4400 9250 4400
 Wire Wire Line
 	9400 4750 9400 4950
 Wire Wire Line
-	9650 4350 9650 4400
-Wire Wire Line
 	9650 4400 9650 4450
-Connection ~ 9250 4400
 Wire Wire Line
 	9400 5150 9400 5500
@@
 Wire Wire Line
 	9400 5500 10150 5500
+Wire Wire Line
+	9250 4300 9250 4350
+Wire Wire Line
+	9650 4300 9650 4350
+$Comp
+L Dual-Mag-Camera-Control-rescue:Si7463DP-ProjectDevices Q?
+U 1 1 60B6F3B7
+P 9450 4350
+AR Path="/60B6F3B7" Ref="Q?"  Part="1"
+AR Path="/5EC85FDF/60B6F3B7" Ref="Q?"  Part="1"
+AR Path="/5EC8F5BD/60B6F3B7" Ref="Q?"  Part="1"
+AR Path="/5EC8F75A/60B6F3B7" Ref="Q?"  Part="1"
+AR Path="/5EC8F75F/60B6F3B7" Ref="Q?"  Part="1"
+AR Path="/5F4A88F1/5F4B61E9/60B6F3B7" Ref="Q?"  Part="1"
+AR Path="/5F4A88F1/5F4C3746/60B6F3B7" Ref="Q?"  Part="1"
+AR Path="/5F4A88F1/5F4C39D3/60B6F3B7" Ref="Q?"  Part="1"
+AR Path="/5F4A88F1/5F4C3D23/60B6F3B7" Ref="Q?"  Part="1"
+AR Path="/5F708A25/60B6F3B7" Ref="Q?"  Part="1"
+AR Path="/5F73D9F1/60B6F3B7" Ref="Q?"  Part="1"
+AR Path="/5F7C3A84/60B6F3B7" Ref="Q?"  Part="1"
+F 0 "Q?" V 9681 4350 50  0000 C CNN
+F 1 "Si7463DP" V 9590 4350 50  0000 C CNN
+F 2 "Package_SO:PowerPAK_SO-8_Single" H 9450 4350 50  0001 C CNN
+F 3 "https://www.vishay.com/docs/72440/si7463dp.pdf" H 9450 4350 50  0001 C CNN
+F 4 "SI7463DP-T1-E3CT-ND" H 9450 4350 50  0001 C CNN "Part Number"
+F 5 "Digikey" H 9450 4350 50  0001 C CNN "Supplier"
+F 6 "https://www.digikey.com/en/products/detail/vishay-siliconix/SI7463DP-T1-E3/1656627" H 9450 4350 50  0001 C CNN "Link"
+	1    9450 4350
+	0    -1   -1   0
+$EndComp
+Wire Wire Line
+	9250 4350 9250 4400
+Connection ~ 9250 4350
+Wire Wire Line
+	9650 4350 9650 4400
+Connection ~ 9650 4350
+Connection ~ 9250 4400
 $EndSCHEMATC
