File: Dual-Mag-Strobe/Dual-Mag-Strobe.kicad_pcb (KiCad board)
At the start: 4 copper layers, 210.4 x 102.5 mm, 182 parts, among them J1 POWER IN, J2 TRIG INPUT, J3 Mating Board Stack, J5 Mating Board Stack, J6 Board Stack, J8 Board Stack, Q1 BSC028N06LS3, Q2 BSC028N06LS3, Q3 BSC028N06LS3, Q4 BSC028N06LS3, Q5 SISS10ADN, Q6 SI7611DN, U1 L1C1-FRD, U10 74AHCT1G14, U11 L1C1-FRD, U12 L1C1-FRD, U13 CreeXD16, U14 CreeXD16, U15 L1C1-FRD, U16 L1C1-FRD, U17 CreeXD16, U18 CreeXD16, U19 LTC4440-5ES6, U2 L1C1-FRD, U20 LTC4440-5ES6, U21 L1C1-FRD, U22 L1C1-FRD, U23 CreeXD16, U24 CreeXD16, U25 L1C1-FRD, U26 L1C1-FRD, U27 CreeXD16, U28 CreeXD16, U29 L1C1-FRD, U3 CreeXD16, U30 L1C1-FRD, U31 CreeXD16, U32 CreeXD16, U33 L1C1-FRD, U34 L1C1-FRD, U35 CreeXD16, U36 CreeXD16, U37 L1C1-FRD, U38 L1C1-FRD, U39 CreeXD16, U4 CreeXD16, U40 CreeXD16, U41 L1C1-FRD, U42 L1C1-FRD, U43 CreeXD16, U44 CreeXD16, U45 L1C1-FRD, U46 L1C1-FRD, U47 CreeXD16, U48 CreeXD16, U49 L1C1-FRD, U5 L1C1-FRD, U50 L1C1-FRD, U51 CreeXD16, U52 CreeXD16, U53 LTC4440-5ES6, U54 LTC4440-5ES6, U55 L1C1-FRD, U56 L1C1-FRD, U57 CreeXD16, U58 CreeXD16, U59 L1C1-FRD, U6 L1C1-FRD, U60 L1C1-FRD, U61 CreeXD16, U62 CreeXD16, U63 74AHCT1G08, U64 74AHCT1G08, U65 L1C1-FRD, U66 L1C1-FRD, U67 CreeXD16, U68 CreeXD16, U69 L1C1-FRD, U7 CreeXD16, U70 L1C1-FRD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

Commit message: updated to KiCAD 6.0
Other:
- net class Default removed
