File: Dual-Mag-Strobe/Dual-Mag-Strobe.sch (KiCad schematic (older format))
At the start: 166 parts, among them J1 POWER IN, J2 TRIG INPUT, J3 Mating Board Stack, J5 Mating Board Stack, J6 Board Stack, J8 Board Stack, Q1 BSC028N06LS3, Q2 BSC028N06LS3, Q3 BSC028N06LS3, Q4 BSC028N06LS3, Q5 SISS10ADN, Q6 SI7611DN, U1 L1C1-FRD, U10 74AHCT1G14, U11 L1C1-FRD, U12 L1C1-FRD, U13 CreeXD16, U14 CreeXD16, U15 L1C1-FRD, U16 L1C1-FRD, U17 CreeXD16, U18 CreeXD16, U19 LTC4440-5ES6, U2 L1C1-FRD, U20 LTC4440-5ES6, U21 L1C1-FRD, U22 L1C1-FRD, U23 CreeXD16, U24 CreeXD16, U25 L1C1-FRD, U26 L1C1-FRD, U27 CreeXD16, U28 CreeXD16, U29 L1C1-FRD, U3 CreeXD16, U30 L1C1-FRD, U31 CreeXD16, U32 CreeXD16, U33 L1C1-FRD, U34 L1C1-FRD, U35 CreeXD16, U36 CreeXD16, U37 L1C1-FRD, U38 L1C1-FRD, U39 CreeXD16, U4 CreeXD16, U40 CreeXD16, U41 L1C1-FRD, U42 L1C1-FRD, U43 CreeXD16, U44 CreeXD16, U45 L1C1-FRD, U46 L1C1-FRD, U47 CreeXD16, U48 CreeXD16, U49 L1C1-FRD, U5 L1C1-FRD, U50 L1C1-FRD, U51 CreeXD16, U52 CreeXD16, U53 LTC4440-5ES6, U54 LTC4440-5ES6, U55 L1C1-FRD, U56 L1C1-FRD, U57 CreeXD16, U58 CreeXD16, U59 L1C1-FRD, U6 L1C1-FRD, U60 L1C1-FRD, U61 CreeXD16, U62 CreeXD16, U63 74AHCT1G08, U64 74AHCT1G08, U65 L1C1-FRD, U66 L1C1-FRD, U67 CreeXD16, U68 CreeXD16, U69 L1C1-FRD, U7 CreeXD16, U70 L1C1-FRD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

Commit message: updated to KiCAD 6.0
Parts:
- C1, C11, C12, C17, C18, C2, C29, C31, C32, C33: symbol CBT-140-Control-rescue:C_Small -> Dual-Mag-Strobe-rescue:C_Small-CBT-140-Control-rescue
- C30: symbol SPC-Control-rescue:C_Small -> Dual-Mag-Strobe-rescue:C_Small-SPC-Control-rescue
- D10, D3, D4, D9: symbol CBT-140-Control-rescue:D -> Dual-Mag-Strobe-rescue:D-CBT-140-Control-rescue
- D14: symbol BUMP-Control-rescue:ZENERsmall-RESCUE-PowerControlBoard-SPC-Control-rescue-DeathStar-rescue -> Dual-Mag-Strobe-rescue:ZENERsmall-RESCUE-PowerControlBoard-SPC-Control-rescue-DeathStar-rescue-BUMP-Control-rescue
- D15, D16, D17: symbol SPC-Control-rescue:D_TVS -> Dual-Mag-Strobe-rescue:D_TVS-SPC-Control-rescue
- D5, D6, D7, D8: symbol CBT-140-Control-rescue:D_Schottky -> Dual-Mag-Strobe-rescue:D_Schottky-CBT-140-Control-rescue
- F2, F3, F4: symbol SPC-Control-rescue:Polyfuse_Small -> Dual-Mag-Strobe-rescue:Polyfuse_Small-SPC-Control-rescue
- Q6: symbol SPC-Control-rescue:SiS443DN -> Dual-Mag-Strobe-rescue:SiS443DN-SPC-Control-rescue
- R10, R4, R6, R8: symbol CBT-140-Control-rescue:R -> Dual-Mag-Strobe-rescue:R-CBT-140-Control-rescue
- R14: symbol BUMP-Control-rescue:Resistor_small-SPC-Control-rescue-DeathStar-rescue -> Dual-Mag-Strobe-rescue:Resistor_small-SPC-Control-rescue-DeathStar-rescue-BUMP-Control-rescue
- R15, R17: symbol SPC-Control-rescue:Resistor_small -> Dual-Mag-Strobe-rescue:Resistor_small-SPC-Control-rescue
- R3, R5, R7, R9: symbol CBT-140-Control-rescue:Resistor_small -> Dual-Mag-Strobe-rescue:Resistor_small-CBT-140-Control-rescue
Changed lines of the file:
@@
 	5650 9150 5350 9150
 $Comp
-L CBT-140-Control-rescue:Resistor_small R9
+L Dual-Mag-Strobe-rescue:Resistor_small-CBT-140-Control-rescue R9
 U 1 1 60007DD3
 P 6650 6450
@@
 	600  4800 600  700
 $Comp
-L SPC-Control-rescue:Polyfuse_Small F3
+L Dual-Mag-Strobe-rescue:Polyfuse_Small-SPC-Control-rescue F3
 U 1 1 60751109
 P 14550 6050
@@
 $EndComp
 $Comp
-L SPC-Control-rescue:D_TVS D16
+L Dual-Mag-Strobe-rescue:D_TVS-SPC-Control-rescue D16
 U 1 1 60751116
 P 14800 6250
@@
 $EndComp
 $Comp
-L BUMP-Control-rescue:ZENERsmall-RESCUE-PowerControlBoard-SPC-Control-rescue-DeathStar-rescue D?
+L Dual-Mag-Strobe-rescue:ZENERsmall-RESCUE-PowerControlBoard-SPC-Control-rescue-DeathStar-rescue-BUMP-Control-rescue D?
 U 1 1 5F7C48C1
 P 13800 1950
@@
 $EndComp
 $Comp
-L BUMP-Control-rescue:Resistor_small-SPC-Control-rescue-DeathStar-rescue R?
+L Dual-Mag-Strobe-rescue:Resistor_small-SPC-Control-rescue-DeathStar-rescue-BUMP-Control-rescue R?
 U 1 1 5F7C48CE
 P 13800 1550
@@
 	13800 1750 13800 1650
 $Comp
-L SPC-Control-rescue:SiS443DN Q?
+L Dual-Mag-Strobe-rescue:SiS443DN-SPC-Control-rescue Q?
 U 1 1 5F4889C4
 P 15400 1500
@@
 $EndComp
 $Comp
-L SPC-Control-rescue:Resistor_small R?
+L Dual-Mag-Strobe-rescue:Resistor_small-SPC-Control-rescue R?
 U 1 1 5F7D2C57
 P 15050 1700
@@
 $EndComp
 $Comp
-L SPC-Control-rescue:Resistor_small R?
+L Dual-Mag-Strobe-rescue:Resistor_small-SPC-Control-rescue R?
 U 1 1 5F7D2C58
 P 15350 2000
@@
 Connection ~ 15600 1350
 $Comp
-L SPC-Control-rescue:C_Small C?
+L Dual-Mag-Strobe-rescue:C_Small-SPC-Control-rescue C?
 U 1 1 5F7D2C5A
 P 14650 1600
@@
 $EndComp
 $Comp
-L SPC-Control-rescue:Polyfuse_Small F2
+L Dual-Mag-Strobe-rescue:Polyfuse_Small-SPC-Control-rescue F2
 U 1 1 60F6C26C
 P 14550 5350
@@
 $EndComp
 $Comp
-L SPC-Control-rescue:D_TVS D15
+L Dual-Mag-Strobe-rescue:D_TVS-SPC-Control-rescue D15
 U 1 1 60F6C279
 P 14800 5550
@@
 GND_PSU
 $Comp
-L SPC-Control-rescue:Polyfuse_Small F4
+L Dual-Mag-Strobe-rescue:Polyfuse_Small-SPC-Control-rescue F4
 U 1 1 6126A313
 P 14550 6750
@@
 $EndComp
 $Comp
-L SPC-Control-rescue:D_TVS D17
+L Dual-Mag-Strobe-rescue:D_TVS-SPC-Control-rescue D17
 U 1 1 6126A320
 P 14800 6950
@@
 	8500 8350 8500 8500
 $Comp
-L CBT-140-Control-rescue:D D?
+L Dual-Mag-Strobe-rescue:D-CBT-140-Control-rescue D?
 U 1 1 61B1B119
 P 8350 7600
@@
 	8600 7600 8500 7600
 $Comp
-L CBT-140-Control-rescue:C_Small C?
+L Dual-Mag-Strobe-rescue:C_Small-CBT-140-Control-rescue C?
 U 1 1 61B1B12B
 P 7950 7600
@@
 Connection ~ 6650 6550
 $Comp
-L CBT-140-Control-rescue:Resistor_small R5
+L Dual-Mag-Strobe-rescue:Resistor_small-CBT-140-Control-rescue R5
 U 1 1 61E49297
 P 5650 6450
@@
 $EndComp
 $Comp
-L CBT-140-Control-rescue:R R?
+L Dual-Mag-Strobe-rescue:R-CBT-140-Control-rescue R?
 U 1 1 61EACDA5
 P 5650 4200
@@
 $EndComp
 $Comp
-L CBT-140-Control-rescue:D_Schottky D?
+L Dual-Mag-Strobe-rescue:D_Schottky-CBT-140-Control-rescue D?
 U 1 1 61EACDB2
 P 5650 2650
@@
 	5650 4600 5350 4600
 $Comp
-L CBT-140-Control-rescue:Resistor_small R7
+L Dual-Mag-Strobe-rescue:Resistor_small-CBT-140-Control-rescue R7
 U 1 1 61EACDC7
 P 6650 1900
@@
 Connection ~ 6650 2000
 $Comp
-L CBT-140-Control-rescue:Resistor_small R3
+L Dual-Mag-Strobe-rescue:Resistor_small-CBT-140-Control-rescue R3
 U 1 1 61EACF3B
 P 5650 1900
@@
 	15600 1350 16100 1350
 $Comp
-L CBT-140-Control-rescue:C_Small C?
+L Dual-Mag-Strobe-rescue:C_Small-CBT-140-Control-rescue C?
 U 1 1 62AAB303
 P 4350 7600
@@
 Connection ~ 4250 7600
 $Comp
-L CBT-140-Control-rescue:D D?
+L Dual-Mag-Strobe-rescue:D-CBT-140-Control-rescue D?
 U 1 1 62AAB81E
 P 3950 7600
@@
 $EndComp
 $Comp
-L CBT-140-Control-rescue:D D?
+L Dual-Mag-Strobe-rescue:D-CBT-140-Control-rescue D?
 U 1 1 62AB03F7
 P 8350 3050
@@
 $EndComp
 $Comp
-L CBT-140-Control-rescue:C_Small C?
+L Dual-Mag-Strobe-rescue:C_Small-CBT-140-Control-rescue C?
 U 1 1 62AB09DC
 P 7950 3050
@@
 Connection ~ 8050 3050
 $Comp
-L CBT-140-Control-rescue:D D?
+L Dual-Mag-Strobe-rescue:D-CBT-140-Control-rescue D?
 U 1 1 62AB106B
 P 3950 3050
@@
 $EndComp
 $Comp
-L CBT-140-Control-rescue:C_Small C?
+L Dual-Mag-Strobe-rescue:C_Small-CBT-140-Control-rescue C?
 U 1 1 62AB16E8
 P 4350 3050
@@
 Connection ~ 4250 3050
 $Comp
-L CBT-140-Control-rescue:R R?
+L Dual-Mag-Strobe-rescue:R-CBT-140-Control-rescue R?
 U 1 1 62AB2218
 P 6650 4200
@@
 $EndComp
 $Comp
-L CBT-140-Control-rescue:R R?
+L Dual-Mag-Strobe-rescue:R-CBT-140-Control-rescue R?
 U 1 1 62AB27F7
 P 6650 8750
@@
 $EndComp
 $Comp
-L CBT-140-Control-rescue:R R?
+L Dual-Mag-Strobe-rescue:R-CBT-140-Control-rescue R?
 U 1 1 62AB3B06
 P 5650 8750
@@
 $EndComp
 $Comp
-L CBT-140-Control-rescue:D_Schottky D?
+L Dual-Mag-Strobe-rescue:D_Schottky-CBT-140-Control-rescue D?
 U 1 1 62AEF8CE
 P 6650 2650
@@
 $EndComp
 $Comp
-L CBT-140-Control-rescue:D_Schottky D?
+L Dual-Mag-Strobe-rescue:D_Schottky-CBT-140-Control-rescue D?
 U 1 1 62AEFDA3
 P 6650 7200
@@
 $EndComp
 $Comp
-L CBT-140-Control-rescue:D_Schottky D?
+L Dual-Mag-Strobe-rescue:D_Schottky-CBT-140-Control-rescue D?
 U 1 1 62AF05D0
 P 5650 7200
@@
 5V_XD16_STROBE
 $Comp
-L CBT-140-Control-rescue:C_Small C?
+L Dual-Mag-Strobe-rescue:C_Small-CBT-140-Control-rescue C?
 U 1 1 62D5DA0F
 P 10100 7800
@@
 	10200 7800 10500 7800
 $Comp
-L CBT-140-Control-rescue:C_Small C?
+L Dual-Mag-Strobe-rescue:C_Small-CBT-140-Control-rescue C?
 U 1 1 62DD2616
 P 10100 3250
@@
 	9350 3250 9350 3400
 $Comp
-L CBT-140-Control-rescue:C_Small C?
+L Dual-Mag-Strobe-rescue:C_Small-CBT-140-Control-rescue C?
 U 1 1 62E0E6F6
 P 2200 3250
@@
 	2950 3250 2950 3400
 $Comp
-L CBT-140-Control-rescue:C_Small C?
+L Dual-Mag-Strobe-rescue:C_Small-CBT-140-Control-rescue C?
 U 1 1 62E4D0B4
 P 2200 7800
@@
 	1200 8000 1150 8000
 $Comp
-L CBT-140-Control-rescue:C_Small C?
+L Dual-Mag-Strobe-rescue:C_Small-CBT-140-Control-rescue C?
 U 1 1 5F7DB7A0
 P 1400 7600
@@
 	1300 7600 1150 7600
 $Comp
-L CBT-140-Control-rescue:C_Small C?
+L Dual-Mag-Strobe-rescue:C_Small-CBT-140-Control-rescue C?
 U 1 1 5F96A7C4
 P 10900 7600
