File: COMMS.kicad_sch (KiCad schematic)
At the start: 38 parts, among them J10 RS-232_2_3, J5 CVS-04TB, J6 CVS-04TB, J7 UART_0_1, J8 UART_2_3, J9 RS-232_0_1

Commit message: Moved Connectors, NEW PTC Footprint
updated ptc footprints to 0603. Relocated GPIO connectors J1-J4
Parts:
- F15, F16, F17, F18, F19, F20, F21, F22, F23, F24, F25, F26, F27, F28, F29, F30: footprint Resistor_SMD:R_1210_3225Metric_Pad1.42x2.65mm_HandSolder -> Resistor_SMD:R_0603_1608Metric_Pad0.98x0.95mm_HandSolder
Changed lines of the file:
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@@
     (property "Reference" "F27" (id 0) (at 240.03 114.935 90))
     (property "Value" "PTC" (id 1) (at 240.03 118.745 90))
-    (property "Footprint" "Resistor_SMD:R_1210_3225Metric_Pad1.42x2.65mm_HandSolder" (id 2) (at 234.95 118.11 0)
+    (property "Footprint" "Resistor_SMD:R_0603_1608Metric_Pad0.98x0.95mm_HandSolder" (id 2) (at 234.95 118.11 0)
       (effects (font (size 1.27 1.27)) (justify left) hide)
     )
@@
     (property "Reference" "F28" (id 0) (at 240.03 135.255 90))
     (property "Value" "PTC" (id 1) (at 240.03 139.065 90))
-    (property "Footprint" "Resistor_SMD:R_1210_3225Metric_Pad1.42x2.65mm_HandSolder" (id 2) (at 234.95 138.43 0)
+    (property "Footprint" "Resistor_SMD:R_0603_1608Metric_Pad0.98x0.95mm_HandSolder" (id 2) (at 234.95 138.43 0)
       (effects (font (size 1.27 1.27)) (justify left) hide)
     )
@@
     (property "Reference" "F29" (id 0) (at 240.03 159.385 90))
     (property "Value" "PTC" (id 1) (at 240.03 163.195 90))
-    (property "Footprint" "Resistor_SMD:R_1210_3225Metric_Pad1.42x2.65mm_HandSolder" (id 2) (at 234.95 162.56 0)
+    (property "Footprint" "Resistor_SMD:R_0603_1608Metric_Pad0.98x0.95mm_HandSolder" (id 2) (at 234.95 162.56 0)
       (effects (font (size 1.27 1.27)) (justify left) hide)
     )
@@
     (property "Reference" "F30" (id 0) (at 240.03 179.705 90))
     (property "Value" "PTC" (id 1) (at 240.03 183.515 90))
-    (property "Footprint" "Resistor_SMD:R_1210_3225Metric_Pad1.42x2.65mm_HandSolder" (id 2) (at 234.95 182.88 0)
+    (property "Footprint" "Resistor_SMD:R_0603_1608Metric_Pad0.98x0.95mm_HandSolder" (id 2) (at 234.95 182.88 0)
       (effects (font (size 1.27 1.27)) (justify left) hide)
     )
@@
     (property "Reference" "F26" (id 0) (at 187.96 179.705 90))
     (property "Value" "PTC" (id 1) (at 187.96 183.515 90))
-    (property "Footprint" "Resistor_SMD:R_1210_3225Metric_Pad1.42x2.65mm_HandSolder" (id 2) (at 182.88 182.88 0)
+    (property "Footprint" "Resistor_SMD:R_0603_1608Metric_Pad0.98x0.95mm_HandSolder" (id 2) (at 182.88 182.88 0)
       (effects (font (size 1.27 1.27)) (justify left) hide)
     )
@@
     (property "Reference" "F25" (id 0) (at 187.96 159.385 90))
     (property "Value" "PTC" (id 1) (at 187.96 163.195 90))
-    (property "Footprint" "Resistor_SMD:R_1210_3225Metric_Pad1.42x2.65mm_HandSolder" (id 2) (at 182.88 162.56 0)
+    (property "Footprint" "Resistor_SMD:R_0603_1608Metric_Pad0.98x0.95mm_HandSolder" (id 2) (at 182.88 162.56 0)
       (effects (font (size 1.27 1.27)) (justify left) hide)
     )
@@
     (property "Reference" "F24" (id 0) (at 187.96 135.255 90))
     (property "Value" "PTC" (id 1) (at 187.96 139.065 90))
-    (property "Footprint" "Resistor_SMD:R_1210_3225Metric_Pad1.42x2.65mm_HandSolder" (id 2) (at 182.88 138.43 0)
+    (property "Footprint" "Resistor_SMD:R_0603_1608Metric_Pad0.98x0.95mm_HandSolder" (id 2) (at 182.88 138.43 0)
       (effects (font (size 1.27 1.27)) (justify left) hide)
     )
@@
     (property "Reference" "F23" (id 0) (at 187.96 114.935 90))
     (property "Value" "PTC" (id 1) (at 187.96 118.745 90))
-    (property "Footprint" "Resistor_SMD:R_1210_3225Metric_Pad1.42x2.65mm_HandSolder" (id 2) (at 182.88 118.11 0)
+    (property "Footprint" "Resistor_SMD:R_0603_1608Metric_Pad0.98x0.95mm_HandSolder" (id 2) (at 182.88 118.11 0)
       (effects (font (size 1.27 1.27)) (justify left) hide)
     )
@@
     (property "Reference" "F19" (id 0) (at 138.43 114.935 90))
     (property "Value" "PTC" (id 1) (at 138.43 118.745 90))
-    (property "Footprint" "Resistor_SMD:R_1210_3225Metric_Pad1.42x2.65mm_HandSolder" (id 2) (at 133.35 118.11 0)
+    (property "Footprint" "Resistor_SMD:R_0603_1608Metric_Pad0.98x0.95mm_HandSolder" (id 2) (at 133.35 118.11 0)
       (effects (font (size 1.27 1.27)) (justify left) hide)
     )
@@
     (property "Reference" "F21" (id 0) (at 138.43 159.385 90))
     (property "Value" "PTC" (id 1) (at 138.43 163.195 90))
-    (property "Footprint" "Resistor_SMD:R_1210_3225Metric_Pad1.42x2.65mm_HandSolder" (id 2) (at 133.35 162.56 0)
+    (property "Footprint" "Resistor_SMD:R_0603_1608Metric_Pad0.98x0.95mm_HandSolder" (id 2) (at 133.35 162.56 0)
       (effects (font (size 1.27 1.27)) (justify left) hide)
     )
@@
     (property "Reference" "F20" (id 0) (at 138.43 135.255 90))
     (property "Value" "PTC" (id 1) (at 138.43 139.065 90))
-    (property "Footprint" "Resistor_SMD:R_1210_3225Metric_Pad1.42x2.65mm_HandSolder" (id 2) (at 133.35 138.43 0)
+    (property "Footprint" "Resistor_SMD:R_0603_1608Metric_Pad0.98x0.95mm_HandSolder" (id 2) (at 133.35 138.43 0)
       (effects (font (size 1.27 1.27)) (justify left) hide)
     )
@@
     (property "Reference" "F22" (id 0) (at 138.43 179.705 90))
     (property "Value" "PTC" (id 1) (at 138.43 183.515 90))
-    (property "Footprint" "Resistor_SMD:R_1210_3225Metric_Pad1.42x2.65mm_HandSolder" (id 2) (at 133.35 182.88 0)
+    (property "Footprint" "Resistor_SMD:R_0603_1608Metric_Pad0.98x0.95mm_HandSolder" (id 2) (at 133.35 182.88 0)
       (effects (font (size 1.27 1.27)) (justify left) hide)
     )
@@
     (property "Reference" "F18" (id 0) (at 97.79 179.705 90))
     (property "Value" "PTC" (id 1) (at 97.79 183.515 90))
-    (property "Footprint" "Resistor_SMD:R_1210_3225Metric_Pad1.42x2.65mm_HandSolder" (id 2) (at 92.71 182.88 0)
+    (property "Footprint" "Resistor_SMD:R_0603_1608Metric_Pad0.98x0.95mm_HandSolder" (id 2) (at 92.71 182.88 0)
       (effects (font (size 1.27 1.27)) (justify left) hide)
     )
@@
     (property "Reference" "F17" (id 0) (at 97.79 159.385 90))
     (property "Value" "PTC" (id 1) (at 97.79 163.195 90))
-    (property "Footprint" "Resistor_SMD:R_1210_3225Metric_Pad1.42x2.65mm_HandSolder" (id 2) (at 92.71 162.56 0)
+    (property "Footprint" "Resistor_SMD:R_0603_1608Metric_Pad0.98x0.95mm_HandSolder" (id 2) (at 92.71 162.56 0)
       (effects (font (size 1.27 1.27)) (justify left) hide)
     )
@@
     (property "Reference" "F16" (id 0) (at 97.79 135.255 90))
     (property "Value" "PTC" (id 1) (at 97.79 139.065 90))
-    (property "Footprint" "Resistor_SMD:R_1210_3225Metric_Pad1.42x2.65mm_HandSolder" (id 2) (at 92.71 138.43 0)
+    (property "Footprint" "Resistor_SMD:R_0603_1608Metric_Pad0.98x0.95mm_HandSolder" (id 2) (at 92.71 138.43 0)
       (effects (font (size 1.27 1.27)) (justify left) hide)
     )
@@
     (property "Reference" "F15" (id 0) (at 97.79 114.935 90))
     (property "Value" "PTC" (id 1) (at 97.79 118.745 90))
-    (property "Footprint" "Resistor_SMD:R_1210_3225Metric_Pad1.42x2.65mm_HandSolder" (id 2) (at 92.71 118.11 0)
-      (effects (font (size 1.27 1.27)) (justify left) hide)
-    )
+    (property "Footprint" "Resistor_SMD:R_0603_1608Metric_Pad0.98x0.95mm_HandSolder" (id 2) (at 92.71 118.11 0)
+      (effects (font (size 1.27 1.27)) (justify left) hide)
+    )
