File: Dual-Mag-Camera-Control.kicad_sch (KiCad schematic)
At the start: 52 parts, among them J1 ~TRIG_IO, J11 PWR_IN_1, J12 PWR_IN_2, J13 STRB_PWR, J14 CAM_COMPUTE_PWR, J15 5V_5A_PWR, J16 5V_2.5A_PWR, J2 TRIG_IO, J3 ADC_DAC, J4 GPIO, U1 D24V10F5, U3 D24V50F5, U4 LowPowerLab-SD-Card, U5 D24V22F5, U8 MoteinoM0

Commit message: Moved Connectors, NEW PTC Footprint
updated ptc footprints to 0603. Relocated GPIO connectors J1-J4
Parts:
- F10, F11, F12, F13, F14, F2, F3, F4, F5, F6, F7, F8, F9: footprint Resistor_SMD:R_1210_3225Metric -> Resistor_SMD:R_0603_1608Metric_Pad0.98x0.95mm_HandSolder
- R5: footprint Resistor_SMD:R_0603_1608Metric_Pad1.05x0.95mm_HandSolder -> Resistor_SMD:R_0603_1608Metric_Pad0.98x0.95mm_HandSolder
